File: hardware/kicad/induction-heater.kicad_pcb (KiCad board)
At the start: 2 copper layers, 99.1 x 76.2 mm, 23 parts, among them J1 Screw_Terminal_01x01, J2 Screw_Terminal_01x01, J3 Screw_Terminal_01x02, Q1 Q_NMOS_DGS, Q2 Q_NMOS_DGS

Commit message: Improved the footprints
Parts:
- R2, R3: footprint Resistor_THT:R_Box_L8.4mm_W2.5mm_P5.08mm -> Package_TO_SOT_THT:TO-220-2_Vertical
- R4, R5: footprint Resistor_THT:R_Axial_DIN0207_L6.3mm_D2.5mm_P10.16mm_Horizontal -> Resistor_THT:R_Axial_DIN0516_L15.5mm_D5.0mm_P5.08mm_Vertical
- moved R2 5.08 mm to (148.6, 30.5), turned to 180 degrees
- moved C1 4.99 mm to (131.4, 76.2)
- moved C2 4.96 mm to (131.4, 50.8)
- moved R4 1.27 mm to (141.0, 48.3), turned to -135 degrees
- moved R5 1.27 mm to (141.0, 78.7), turned to 135 degrees
- moved D4 1.27 mm to (152.4, 83.8)
- moved R3 0.31 mm to (143.5, 96.8)
Routing:
- net Net-(D2-Pad1): track 60.3 -> 55.8 mm
- net Net-(D1-Pad1): track 48.1 -> 49.2 mm
