File: hardware/kicad/induction-heater.kicad_pcb (KiCad board)
At the start: 2 copper layers, 99.1 x 76.2 mm, 23 parts, among them J1 Screw_Terminal_01x01, J2 Screw_Terminal_01x01, J3 Screw_Terminal_01x02, Q1 Q_NMOS_DGS, Q2 Q_NMOS_DGS

Commit message: Finishing up
Routing:
- net Net-(D1-Pad1): track 42.5 -> 48.6 mm
- net Net-(D2-Pad1): track 54.6 -> 52.8 mm
- net /out_l: track 30.3 -> 31.3 mm
Other:
- board text added: "Induction heater V2 2022 Dion Dokter Carmine Crystal"
Changed lines of the file:
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@@
     (descr "TO-220-2, Vertical, RM 5.08mm, see https://www.centralsemi.com/PDFS/CASE/TO-220-2PD.PDF")
     (tags "TO-220-2 Vertical RM 5.08mm")
+    (property "MPN" "AP851470RJ")
     (property "Max V" "420")
     (property "Sheetfile" "induction-heater.kicad_sch")
@@
     (descr "Resistor, Axial_DIN0516 series, Axial, Vertical, pin pitch=5.08mm, 2W, length*diameter=15.5*5mm^2, http://cdn-reichelt.de/documents/datenblatt/B400/1_4W%23YAG.pdf")
     (tags "Resistor Axial_DIN0516 series Axial Vertical pin pitch 5.08mm 2W length 15.5mm diameter 5mm")
+    (property "MPN" "ROX3SJ10K")
     (property "Max V" "350")
     (property "Sheetfile" "induction-heater.kicad_sch")
@@
     (descr "TO-220-2, Vertical, RM 5.08mm, see https://www.centralsemi.com/PDFS/CASE/TO-220-2PD.PDF")
     (tags "TO-220-2 Vertical RM 5.08mm")
+    (property "MPN" "AP851470RJ")
     (property "Max V" "420")
     (property "Sheetfile" "induction-heater.kicad_sch")
@@
     (descr "Resistor, Axial_DIN0516 series, Axial, Vertical, pin pitch=5.08mm, 2W, length*diameter=15.5*5mm^2, http://cdn-reichelt.de/documents/datenblatt/B400/1_4W%23YAG.pdf")
     (tags "Resistor Axial_DIN0516 series Axial Vertical pin pitch 5.08mm 2W length 15.5mm diameter 5mm")
+    (property "MPN" "ROX3SJ10K")
     (property "Max V" "350")
     (property "Sheetfile" "induction-heater.kicad_sch")
@@
   )
   (gr_rect (start 226.06 101.6) (end 127 25.4) (layer "Edge.Cuts") (width 0.1) (fill none))
+  (gr_text "Induction heater V2 2022\nDion Dokter\nCarmine Crystal" (at 161.925 31.115 180) (layer "B.SilkS")
+    (effects (font (size 1.5 1.5) (thickness 0.3)) (justify left mirror))
+  )
   (gr_text "Vcc" (at 129.54 55.88) (layer "F.SilkS")
     (effects (font (size 1 1) (thickness 0.15)))
@@
     (effects (font (size 1 1) (thickness 0.15)))
   )
-  (segment (start 143.51 37.775) (end 143.51 52.07) (width 2.5) (layer "F.Cu") (net 3))
   (segment (start 152.62 52.07) (end 154.94 49.75) (width 2.5) (layer "F.Cu") (net 3))
+  (segment (start 143.51 41.91) (end 144.78 43.18) (width 2.5) (layer "F.Cu") (net 3))
+  (segment (start 144.78 50.8) (end 143.51 52.07) (width 2.5) (layer "F.Cu") (net 3))
+  (segment (start 143.51 37.775) (end 143.51 41.91) (width 2.5) (layer "F.Cu") (net 3))
   (segment (start 143.51 52.07) (end 152.62 52.07) (width 2.5) (layer "F.Cu") (net 3))
+  (segment (start 144.78 43.18) (end 144.78 50.8) (width 2.5) (layer "F.Cu") (net 3))
   (segment (start 215.9 38.1) (end 218.44 35.56) (width 2.5) (layer "B.Cu") (net 3))
   (segment (start 152.62 74.93) (end 143.51 74.93) (width 2.5) (layer "F.Cu") (net 4))
@@
   (segment (start 152.0425 89.225) (end 156.21 85.0575) (width 2.5) (layer "F.Cu") (net 4))
   (segment (start 156.21 78.52) (end 154.94 77.25) (width 2.5) (layer "F.Cu") (net 4))
+  (segment (start 140.97 53.975) (end 139.7 55.245) (width 0.8) (layer "F.Cu") (net 5))
   (segment (start 139.7 43.18) (end 139.7 36.83) (width 0.8) (layer "F.Cu") (net 5))
   (segment (start 146.05 35.56) (end 146.05 37.775) (width 0.8) (layer "F.Cu") (net 5))
@@
   (segment (start 144.785 34.29) (end 144.78 34.29) (width 0.8) (layer "F.Cu") (net 5))
   (segment (start 148.595 30.48) (end 144.785 34.29) (width 0.8) (layer "F.Cu") (net 5))
+  (segment (start 139.7 46.99) (end 140.97 48.26) (width 0.8) (layer "F.Cu") (net 5))
   (segment (start 144.78 34.29) (end 146.05 35.56) (width 0.8) (layer "F.Cu") (net 5))
+  (segment (start 140.97 48.26) (end 140.97 53.975) (width 0.8) (layer "F.Cu") (net 5))
+  (segment (start 139.7 43.18) (end 139.7 46.99) (width 0.8) (layer "F.Cu") (net 5))
   (segment (start 142.24 34.29) (end 144.78 34.29) (width 0.8) (layer "F.Cu") (net 5))
   (segment (start 139.7 63.5) (end 143.51 67.31) (width 0.8) (layer "F.Cu") (net 5))
-  (segment (start 139.7 48.26) (end 139.7 63.5) (width 0.8) (layer "F.Cu") (net 5))
+  (segment (start 139.7 55.245) (end 139.7 63.5) (width 0.8) (layer "F.Cu") (net 5))
   (segment (start 147.32 83.82) (end 146.05 85.09) (width 0.8) (layer "F.Cu") (net 6))
+  (segment (start 143.1 71.12) (end 146.05 71.12) (width 0.8) (layer "F.Cu") (net 6))
+  (segment (start 147.32 69.85) (end 147.32 63.5) (width 0.8) (layer "F.Cu") (net 6))
   (segment (start 146.05 85.09) (end 146.05 89.225) (width 0.8) (layer "F.Cu") (net 6))
-  (segment (start 143.1 71.12) (end 146.05 71.12) (width 0.8) (layer "F.Cu") (net 6))
+  (segment (start 140.97 73.25) (end 143.1 71.12) (width 0.8) (layer "F.Cu") (net 6))
+  (segment (start 146.05 89.225) (end 146.05 92.71) (width 0.8) (layer "F.Cu") (net 6))
+  (segment (start 147.32 83.82) (end 142.24 78.74) (width 0.8) (layer "F.Cu") (net 6))
+  (segment (start 147.32 63.5) (end 143.51 59.69) (width 0.8) (layer "F.Cu") (net 6))
   (segment (start 146.05 71.12) (end 147.32 69.85) (width 0.8) (layer "F.Cu") (net 6))
-  (segment (start 139.7 78.74) (end 142.24 78.74) (width 0.8) (layer "F.Cu") (net 6))
-  (segment (start 146.05 89.225) (end 146.05 92.71) (width 0.8) (layer "F.Cu") (net 6))
-  (segment (start 147.32 83.82) (end 146.05 82.55) (width 0.8) (layer "F.Cu") (net 6))
-  (segment (start 142.24 78.74) (end 146.05 82.55) (width 0.8) (layer "F.Cu") (net 6))
-  (segment (start 139.7 74.52) (end 143.1 71.12) (width 0.8) (layer "F.Cu") (net 6))
   (segment (start 146.05 92.71) (end 148.595 95.255) (width 0.8) (layer "F.Cu") (net 6))
   (segment (start 152.4 83.82) (end 147.32 83.82) (width 0.8) (layer "F.Cu") (net 6))
-  (segment (start 147.32 69.85) (end 147.32 63.5) (width 0.8) (layer "F.Cu") (net 6))
+  (segment (start 140.97 78.74) (end 140.97 73.25) (width 0.8) (layer "F.Cu") (net 6))
+  (segment (start 142.24 78.74) (end 140.97 78.74) (width 0.8) (layer "F.Cu") (net 6))
   (segment (start 148.595 95.255) (end 148.595 96.52) (width 0.8) (layer "F.Cu") (net 6))
-  (segment (start 139.7 78.74) (end 139.7 74.52) (width 0.8) (layer "F.Cu") (net 6))
-  (segment (start 147.32 63.5) (end 143.51 59.69) (width 0.8) (layer "F.Cu") (net 6))
   (zone (net 4) (net_name "/out_r") (layers F&B.Cu) (hatch edge 0.508)
     (priority 1)

Commit message: Fixed resistor pin assignment on board
Routing:
- net Net-(D1-Pad1): track 48.6 -> 46.9 mm
Changed lines of the file:
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@@
   (segment (start 156.21 78.52) (end 154.94 77.25) (width 2.5) (layer "F.Cu") (net 4))
   (segment (start 140.97 53.975) (end 139.7 55.245) (width 0.8) (layer "F.Cu") (net 5))
-  (segment (start 139.7 43.18) (end 139.7 36.83) (width 0.8) (layer "F.Cu") (net 5))
   (segment (start 146.05 35.56) (end 146.05 37.775) (width 0.8) (layer "F.Cu") (net 5))
-  (segment (start 139.7 36.83) (end 142.24 34.29) (width 0.8) (layer "F.Cu") (net 5))
   (segment (start 144.785 34.29) (end 144.78 34.29) (width 0.8) (layer "F.Cu") (net 5))
-  (segment (start 148.595 30.48) (end 144.785 34.29) (width 0.8) (layer "F.Cu") (net 5))
+  (segment (start 143.51 30.48) (end 143.51 33.02) (width 0.8) (layer "F.Cu") (net 5))
   (segment (start 139.7 46.99) (end 140.97 48.26) (width 0.8) (layer "F.Cu") (net 5))
   (segment (start 144.78 34.29) (end 146.05 35.56) (width 0.8) (layer "F.Cu") (net 5))
   (segment (start 140.97 48.26) (end 140.97 53.975) (width 0.8) (layer "F.Cu") (net 5))
   (segment (start 139.7 43.18) (end 139.7 46.99) (width 0.8) (layer "F.Cu") (net 5))
-  (segment (start 142.24 34.29) (end 144.78 34.29) (width 0.8) (layer "F.Cu") (net 5))
   (segment (start 139.7 63.5) (end 143.51 67.31) (width 0.8) (layer "F.Cu") (net 5))
+  (segment (start 139.7 36.83) (end 143.51 33.02) (width 0.8) (layer "F.Cu") (net 5))
+  (segment (start 139.7 43.18) (end 139.7 36.83) (width 0.8) (layer "F.Cu") (net 5))
+  (segment (start 143.51 33.02) (end 144.78 34.29) (width 0.8) (layer "F.Cu") (net 5))
   (segment (start 139.7 55.245) (end 139.7 63.5) (width 0.8) (layer "F.Cu") (net 5))
   (segment (start 147.32 83.82) (end 146.05 85.09) (width 0.8) (layer "F.Cu") (net 6))

Commit message: V2 done. Also added a new simulation design for a possible v3
Parts:
- Q1, Q2: value Q_NMOS_DGS -> Q_NMOS_GDS
- moved D1 7.62 mm to (143.5, 74.9), turned to 90 degrees
- moved D2 6.98 mm to (143.5, 52.7), turned to -90 degrees
- moved R4 2.84 mm to (138.4, 49.5), turned to -90 degrees
- moved R5 2.84 mm to (138.4, 77.5), turned to 90 degrees
Connections:
- D1 pad 1: Net-(D1-Pad1) -> /out_r
- D1 pad 2: /out_r -> Net-(D3-Pad1)
- D2 pad 1: Net-(D2-Pad1) -> /out_l
- D2 pad 2: /out_l -> Net-(D4-Pad1)
- D3 pad 1: Net-(D1-Pad1) -> Net-(D3-Pad1)
- D4 pad 1: Net-(D2-Pad1) -> Net-(D4-Pad1)
- Q1 pad 1: /out_l -> Net-(D3-Pad1)
- Q1 pad 2: Net-(D1-Pad1) -> /out_l
- Q2 pad 1: /out_r -> Net-(D4-Pad1)
- Q2 pad 2: Net-(D2-Pad1) -> /out_r
- R2 pad 2: Net-(D1-Pad1) -> Net-(D3-Pad1)
- R3 pad 2: Net-(D2-Pad1) -> Net-(D4-Pad1)
- R4 pad 1: Net-(D1-Pad1) -> Net-(D3-Pad1)
- R5 pad 1: Net-(D2-Pad1) -> Net-(D4-Pad1)
Routing:
- net Net-(D4-Pad1): track 0.00 -> 64.3 mm
- net Net-(D2-Pad1): track 52.8 -> 0.00 mm
- net Net-(D1-Pad1): track 46.9 -> 0.00 mm
- net Net-(D3-Pad1): track 0.00 -> 41.0 mm
- net GND: track 0.00 -> 18.3 mm, vias 0 -> 2
- net /out_r: track 30.1 -> 27.7 mm
Other:
- outline, holes or cut-outs redrawn
- board text added: "Induction heater V2 2023 Dion Dokter Carmine Crystal"
- board text removed: "Induction heater V2 2022 Dion Dokter Carmine Crystal"
