File: hardware/kicad/induction-heater.kicad_sch (KiCad schematic)
At the start: 23 parts, among them J1 Screw_Terminal_01x01, J2 Screw_Terminal_01x01, J3 Screw_Terminal_01x02, Q1 Q_NMOS_DGS, Q2 Q_NMOS_DGS

Commit message: Improved the footprints
Parts:
- R2, R3: footprint Resistor_THT:R_Box_L8.4mm_W2.5mm_P5.08mm -> Package_TO_SOT_THT:TO-220-2_Vertical
- R4, R5: footprint Resistor_THT:R_Axial_DIN0207_L6.3mm_D2.5mm_P10.16mm_Horizontal -> Resistor_THT:R_Axial_DIN0516_L15.5mm_D5.0mm_P5.08mm_Vertical
Changed lines of the file:
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@@
     (property "Reference" "R3" (id 0) (at 88.9 69.85 90))
     (property "Value" "470" (id 1) (at 88.9 72.39 90))
-    (property "Footprint" "Resistor_THT:R_Box_L8.4mm_W2.5mm_P5.08mm" (id 2) (at 88.9 77.978 90)
+    (property "Footprint" "Package_TO_SOT_THT:TO-220-2_Vertical" (id 2) (at 88.9 77.978 90)
       (effects (font (size 1.27 1.27)) hide)
     )
@@
       (effects (font (size 1.27 1.27)) (justify left))
     )
-    (property "Footprint" "Resistor_THT:R_Axial_DIN0207_L6.3mm_D2.5mm_P10.16mm_Horizontal" (id 2) (at 97.282 82.55 90)
+    (property "Footprint" "Resistor_THT:R_Axial_DIN0516_L15.5mm_D5.0mm_P5.08mm_Vertical" (id 2) (at 97.282 82.55 90)
       (effects (font (size 1.27 1.27)) hide)
     )
@@
     (property "Reference" "R2" (id 0) (at 88.9 31.75 90))
     (property "Value" "470" (id 1) (at 88.9 34.29 90))
-    (property "Footprint" "Resistor_THT:R_Box_L8.4mm_W2.5mm_P5.08mm" (id 2) (at 88.9 39.878 90)
+    (property "Footprint" "Package_TO_SOT_THT:TO-220-2_Vertical" (id 2) (at 88.9 39.878 90)
       (effects (font (size 1.27 1.27)) hide)
     )
@@
       (effects (font (size 1.27 1.27)) (justify left))
     )
-    (property "Footprint" "Resistor_THT:R_Axial_DIN0207_L6.3mm_D2.5mm_P10.16mm_Horizontal" (id 2) (at 97.282 44.45 90)
+    (property "Footprint" "Resistor_THT:R_Axial_DIN0516_L15.5mm_D5.0mm_P5.08mm_Vertical" (id 2) (at 97.282 44.45 90)
       (effects (font (size 1.27 1.27)) hide)
     )
@@
     )
     (path "/eaf5dfa2-8175-42ae-a65a-8e2e940ed4eb"
-      (reference "R2") (unit 1) (value "470") (footprint "Resistor_THT:R_Box_L8.4mm_W2.5mm_P5.08mm")
+      (reference "R2") (unit 1) (value "470") (footprint "Package_TO_SOT_THT:TO-220-2_Vertical")
     )
     (path "/1bc27ce4-f902-44ff-b3ec-5a09b750c013"
-      (reference "R3") (unit 1) (value "470") (footprint "Resistor_THT:R_Box_L8.4mm_W2.5mm_P5.08mm")
+      (reference "R3") (unit 1) (value "470") (footprint "Package_TO_SOT_THT:TO-220-2_Vertical")
     )
     (path "/f74691b4-ab73-45d2-adb2-a73aca070029"
-      (reference "R4") (unit 1) (value "10K") (footprint "Resistor_THT:R_Axial_DIN0207_L6.3mm_D2.5mm_P10.16mm_Horizontal")
+      (reference "R4") (unit 1) (value "10K") (footprint "Resistor_THT:R_Axial_DIN0516_L15.5mm_D5.0mm_P5.08mm_Vertical")
     )
     (path "/799c8382-e657-4e5c-be05-62a7733f4321"
-      (reference "R5") (unit 1) (value "10K") (footprint "Resistor_THT:R_Axial_DIN0207_L6.3mm_D2.5mm_P10.16mm_Horizontal")
-    )
-  )
+      (reference "R5") (unit 1) (value "10K") (footprint "Resistor_THT:R_Axial_DIN0516_L15.5mm_D5.0mm_P5.08mm_Vertical")
+    )
+  )
