File: hardware/kicad/induction-heater.kicad_sch (KiCad schematic)
At the start: 23 parts, among them J1 Screw_Terminal_01x01, J2 Screw_Terminal_01x01, J3 Screw_Terminal_01x02, Q1 Q_NMOS_DGS, Q2 Q_NMOS_DGS

Commit message: V2 done. Also added a new simulation design for a possible v3
Parts:
- D1, D2: symbol pspice:DIODE -> Diode:1N4005
- Q1, Q2: value Q_NMOS_DGS -> Q_NMOS_GDS; symbol Device:Q_NMOS_DGS -> Device:Q_NMOS_GDS
Connections:
- net out_l: now also D2.1 (K), Q1.2 (D); no longer D2.2 (A), Q1.1 (D)
- net out_r: now also D1.1 (K), Q2.2 (D); no longer D1.2 (A), Q2.1 (D)
- net at D4.1 (K), R3.2, R5.1: now also D2.2 (A), Q2.1 (G); no longer D2.1 (K), Q2.2 (G)
- net at D3.1 (K), R2.2, R4.1: now also D1.2 (A), Q1.1 (G); no longer D1.1 (K), Q1.2 (G)
Changed lines of the file:
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@@
     (stroke (width 0) (type default) (color 0 0 0 0))
   )
-  (wire (pts (xy 111.76 60.96) (xy 111.76 63.5))
+  (wire (pts (xy 111.76 60.96) (xy 111.76 64.77))
     (stroke (width 0) (type default) (color 0 0 0 0))
   )
@@
     (stroke (width 0) (type default) (color 0 0 0 0))
   )
-  (wire (pts (xy 111.76 22.86) (xy 111.76 25.4))
+  (wire (pts (xy 111.76 22.86) (xy 111.76 26.67))
     (stroke (width 0) (type default) (color 0 0 0 0))
   )
@@
     (stroke (width 0) (type default) (color 0 0 0 0))
   )
-  (wire (pts (xy 111.76 73.66) (xy 111.76 76.2))
-    (stroke (width 0) (type default) (color 0 0 0 0))
-  )
-  (wire (pts (xy 111.76 35.56) (xy 111.76 38.1))
+  (wire (pts (xy 111.76 72.39) (xy 111.76 76.2))
+    (stroke (width 0) (type default) (color 0 0 0 0))
+  )
+  (wire (pts (xy 111.76 34.29) (xy 111.76 38.1))
     (stroke (width 0) (type default) (color 0 0 0 0))
   )
@@
     (pin "1")
   )
-  (symbol (lib_id "Device:Q_NMOS_DGS") (at 134.62 76.2 0) (unit 1)
+  (symbol (lib_id "Device:Q_NMOS_GDS") (at 134.62 76.2 0) (unit 1)
     (in_bom yes) (on_board yes) (fields_autoplaced)
     (property "Reference" "Q2" (id 0) (at 140.97 74.9299 0)
       (effects (font (size 1.27 1.27)) (justify left))
     )
-    (property "Value" "Q_NMOS_DGS" (id 1) (at 140.97 77.4699 0)
+    (property "Value" "Q_NMOS_GDS" (id 1) (at 140.97 77.4699 0)
       (effects (font (size 1.27 1.27)) (justify left))
     )
@@
       (effects (font (size 1.27 1.27)) hide)
     )
-    (property "Datasheet" "https://nl.mouser.com/datasheet/2/308/NTP067N65S3H_D-2037433.pdf" (id 3) (at 134.62 76.2 0)
+    (property "Datasheet" "~" (id 3) (at 134.62 76.2 0)
       (effects (font (size 1.27 1.27)) hide)
     )
@@
     (pin "2")
   )
-  (symbol (lib_id "pspice:DIODE") (at 111.76 30.48 90) (unit 1)
-    (in_bom yes) (on_board yes) (fields_autoplaced)
-    (property "Reference" "D1" (id 0) (at 115.57 29.2099 90)
-      (effects (font (size 1.27 1.27)) (justify right))
-    )
-    (property "Value" "DIODE" (id 1) (at 115.57 31.7499 90)
-      (effects (font (size 1.27 1.27)) (justify right))
-    )
-    (property "Footprint" "Diode_THT:D_DO-41_SOD81_P7.62mm_Horizontal" (id 2) (at 111.76 30.48 0)
+  (symbol (lib_id "Diode:1N4005") (at 111.76 30.48 270) (unit 1)
+    (in_bom yes) (on_board yes) (fields_autoplaced)
+    (property "Reference" "D1" (id 0) (at 114.3 29.2099 90)
+      (effects (font (size 1.27 1.27)) (justify left))
+    )
+    (property "Value" "DIODE" (id 1) (at 114.3 31.7499 90)
+      (effects (font (size 1.27 1.27)) (justify left))
+    )
+    (property "Footprint" "Diode_THT:D_DO-41_SOD81_P7.62mm_Horizontal" (id 2) (at 107.315 30.48 0)
       (effects (font (size 1.27 1.27)) hide)
     )
@@
     (pin "2")
   )
-  (symbol (lib_id "Device:Q_NMOS_DGS") (at 134.62 38.1 0) (unit 1)
+  (symbol (lib_id "Device:Q_NMOS_GDS") (at 134.62 38.1 0) (unit 1)
     (in_bom yes) (on_board yes) (fields_autoplaced)
     (property "Reference" "Q1" (id 0) (at 140.97 36.8299 0)
       (effects (font (size 1.27 1.27)) (justify left))
     )
-    (property "Value" "Q_NMOS_DGS" (id 1) (at 140.97 39.3699 0)
+    (property "Value" "Q_NMOS_GDS" (id 1) (at 140.97 39.3699 0)
       (effects (font (size 1.27 1.27)) (justify left))
     )
@@
       (effects (font (size 1.27 1.27)) hide)
     )
-    (property "Datasheet" "https://nl.mouser.com/datasheet/2/308/NTP067N65S3H_D-2037433.pdf" (id 3) (at 134.62 38.1 0)
+    (property "Datasheet" "~" (id 3) (at 134.62 38.1 0)
       (effects (font (size 1.27 1.27)) hide)
     )
@@
     (pin "1")
   )
-  (symbol (lib_id "pspice:DIODE") (at 111.76 68.58 90) (unit 1)
-    (in_bom yes) (on_board yes) (fields_autoplaced)
-    (property "Reference" "D2" (id 0) (at 115.57 67.3099 90)
-      (effects (font (size 1.27 1.27)) (justify right))
-    )
-    (property "Value" "DIODE" (id 1) (at 115.57 69.8499 90)
-      (effects (font (size 1.27 1.27)) (justify right))
-    )
-    (property "Footprint" "Diode_THT:D_DO-41_SOD81_P7.62mm_Horizontal" (id 2) (at 111.76 68.58 0)
+  (symbol (lib_id "Diode:1N4005") (at 111.76 68.58 270) (unit 1)
+    (in_bom yes) (on_board yes) (fields_autoplaced)
+    (property "Reference" "D2" (id 0) (at 114.3 67.3099 90)
+      (effects (font (size 1.27 1.27)) (justify left))
+    )
+    (property "Value" "DIODE" (id 1) (at 114.3 69.8499 90)
+      (effects (font (size 1.27 1.27)) (justify left))
+    )
+    (property "Footprint" "Diode_THT:D_DO-41_SOD81_P7.62mm_Horizontal" (id 2) (at 107.315 68.58 0)
       (effects (font (size 1.27 1.27)) hide)
     )
@@
     )
     (path "/768274d5-d1de-4b65-9750-67cf245514d4"
-      (reference "Q1") (unit 1) (value "Q_NMOS_DGS") (footprint "Package_TO_SOT_THT:TO-220-3_Vertical")
+      (reference "Q1") (unit 1) (value "Q_NMOS_GDS") (footprint "Package_TO_SOT_THT:TO-220-3_Vertical")
     )
     (path "/14cf6713-8d1e-4190-9cf8-f2f74832fb89"
-      (reference "Q2") (unit 1) (value "Q_NMOS_DGS") (footprint "Package_TO_SOT_THT:TO-220-3_Vertical")
+      (reference "Q2") (unit 1) (value "Q_NMOS_GDS") (footprint "Package_TO_SOT_THT:TO-220-3_Vertical")
     )
     (path "/eaf5dfa2-8175-42ae-a65a-8e2e940ed4eb"
